Commit message: Gazebo

File: Simulation/sim_ws/src/duanbot_description/urdf/duanbot/actuator/caster.urdf.xacro (robot description, xacro)
@@ -1,4 +1,5 @@
 <?xml version="1.0"?>
 <robot xmlns:xacro="http://www.ros.org/wiki/xacro">
+<xacro:include filename="$(find duanbot_description)/urdf/duanbot/common_inertia.xacro"/>
     <xacro:macro name="caster_xacro" params="caster_name xyz">
         <!-- 机器人的IMU部件，惯性测量传感器 -->
@@ -18,4 +19,18 @@
                 </material>
             </visual>
+            <collision>
+                <!-- 沿着自己几何中心的偏移和旋转 -->
+                <origin xyz="0.0 0.0 0.0" rpy="1.57079 0.0 0.0"/>
+                <!-- 几何形状 -->
+                <geometry>
+                    <!-- 圆柱体 radius 半径 0.10m  高度 0.12m-->
+                    <sphere radius="0.016"/>
+                </geometry>
+                <!-- 材质颜色 -->
+                <material name="yellow">
+                    <color rgba="1.0 1.0 0.0 0.8"/>
+                </material>
+            </collision>
+            <xacro:sphere_inertia m="0.05" r="0.016" />
         </link>
         <!-- 机器人的关节，用于组合机器人的部件 -->
@@ -27,4 +42,10 @@
             <axis xyz="0 1 0"/>
         </joint>
+        <gazebo reference="${caster_name}_link">
+            <mu1 value="0.0"/>
+            <mu2 value="0.0"/>
+            <kp value="1000000000.0"/>
+            <kd value="1.0"/>
+        </gazebo>
     </xacro:macro>
 </robot>

File: Simulation/sim_ws/src/duanbot_description/urdf/duanbot/actuator/wheel.urdf.xacro (robot description, xacro)
@@ -1,4 +1,5 @@
 <?xml version="1.0"?>
 <robot xmlns:xacro="http://www.ros.org/wiki/xacro">
+<xacro:include filename="$(find duanbot_description)/urdf/duanbot/common_inertia.xacro"/>
     <xacro:macro name="wheel_xacro" params="wheel_name xyz">
         <!-- 机器人的IMU部件，惯性测量传感器 -->
@@ -18,4 +19,18 @@
                 </material>
             </visual>
+            <collision>
+                <!-- 沿着自己几何中心的偏移和旋转 -->
+                <origin xyz="0.0 0.0 0.0" rpy="1.57079 0.0 0.0"/>
+                <!-- 几何形状 -->
+                <geometry>
+                    <!-- 圆柱体 radius 半径 0.10m  高度 0.12m-->
+                    <cylinder radius="0.032" length="0.04"/>
+                </geometry>
+                <!-- 材质颜色 -->
+                <material name="yellow">
+                    <color rgba="1.0 1.0 0.0 0.8"/>
+                </material>
+            </collision>
+            <xacro:cylinder_inertia m="0.05" r="0.032" h="0.04" />
         </link>
         <!-- 机器人的关节，用于组合机器人的部件 -->
@@ -27,4 +42,10 @@
             <axis xyz="0 1 0"/>
         </joint>
+        <gazebo reference="${wheel_name}_link">
+            <mu1 value="20.0"/>
+            <mu2 value="20.0"/>
+            <kp value="1000000000.0"/>
+            <kd value="1.0"/>
+        </gazebo>
     </xacro:macro>
 </robot>

File: Simulation/sim_ws/src/duanbot_description/urdf/duanbot/base.urdf.xacro (robot description, xacro)
@@ -1,5 +1,8 @@
 <?xml version="1.0"?>
 <robot xmlns:xacro="http://www.ros.org/wiki/xacro">
+    <!-- 像引入头文件一样 引入惯性相关 -->
+    <xacro:include filename="$(find duanbot_description)/urdf/duanbot/common_inertia.xacro"/>
     <xacro:macro name="base_xacro" params="length radius">
+        <link name="base_footprint"/>
         <link name="base_link">
             <!-- 部件的外观描述 -->
@@ -17,5 +20,25 @@
                 </material>
             </visual>
+            <collision>
+                <!-- 沿着自己几何中心的偏移和旋转 -->
+                <origin xyz="0.0 0.0 0.0" rpy="0.0 0.0 0.0"/>
+                <!-- 几何形状 -->
+                <geometry>
+                    <!-- 圆柱体 radius 半径 0.10m  高度 0.12m-->
+                    <cylinder radius="${radius}" length="${length}"/>
+                </geometry>
+                <!-- 材质颜色 -->
+                <material name="white">
+                    <color rgba="1.0 1.0 1.0 0.5"/>
+                </material>
+            </collision>
+            <!-- 添加好惯性矩阵 -->
+            <xacro:cylinder_inertia m="1.0" r="${radius}" h="${length}" />
         </link>
+        <joint name="base_joint" type="fixed">
+            <parent link="base_footprint"/>
+            <child link="base_link"/>
+            <origin xyz="0.0 0.0 ${length/2.0+0.032-0.001}" rpy="0 0 0"/>
+        </joint>
     </xacro:macro>
 </robot>

File: Simulation/sim_ws/src/duanbot_description/urdf/duanbot/duanbot.urdf.xacro (robot description, xacro)
@@ -10,6 +10,8 @@
 <xacro:include filename="$(find duanbot_description)/urdf/duanbot/actuator/wheel.urdf.xacro"/>
 <xacro:include filename="$(find duanbot_description)/urdf/duanbot/actuator/caster.urdf.xacro"/>
+<!-- 插件 -->
+<xacro:include filename="$(find duanbot_description)/urdf/duanbot/plugins/gazebo_control_plugin.xacro"/>
 <xacro:base_xacro length="0.12" radius="0.10" />
-<xacro:imu_xacro xyz="0.0 0.0 0.2" />
+<xacro:imu_xacro xyz="0.0 0.0 0.02" />
 <xacro:camera_xacro xyz="0.10 0.0 0.075" />
 <xacro:laser_xacro xyz="0.0 0.0 0.10" />
@@ -18,3 +20,4 @@
 <xacro:caster_xacro caster_name="front_caster" xyz="0.08 0.0 -0.076"/>
 <xacro:caster_xacro caster_name="back_caster" xyz="-0.08 0.0 -0.076"/>
+<xacro:gazebo_control_plugin />
 </robot>

File: Simulation/sim_ws/src/duanbot_description/urdf/duanbot/sensor/camera.urdf.xacro (robot description, xacro)
@@ -1,4 +1,5 @@
 <?xml version="1.0"?>
 <robot xmlns:xacro="http://www.ros.org/wiki/xacro">
+<xacro:include filename="$(find duanbot_description)/urdf/duanbot/common_inertia.xacro"/>
     <xacro:macro name="camera_xacro" params="xyz">
         <link name="camera_link">
@@ -16,4 +17,17 @@
                 </material>
             </visual>
+            <collision>
+                <!-- 沿着自己几何中心的偏移和旋转 -->
+                <origin xyz="0.0 0.0 0.0" rpy="0.0 0.0 0.0"/>
+                <!-- 几何形状 -->
+                <geometry>
+                    <box size="0.02 0.10 0.02"/>
+                </geometry>
+                <!-- 材质颜色 -->
+                <material name="black">
+                    <color rgba="0.0 0.0 0.0 0.5"/>
+                </material>
+            </collision>
+            <xacro:box_inertia m="0.1" w="0.02" h="0.10" d="0.02" />
         </link>
         <!-- 机器人的关节，用于组合机器人的部件 -->

File: Simulation/sim_ws/src/duanbot_description/urdf/duanbot/sensor/imu.urdf.xacro (robot description, xacro)
@@ -1,4 +1,5 @@
 <?xml version="1.0"?>
 <robot xmlns:xacro="http://www.ros.org/wiki/xacro">
+<xacro:include filename="$(find duanbot_description)/urdf/duanbot/common_inertia.xacro"/>
     <xacro:macro name="imu_xacro" params="xyz">
         <!-- 机器人的IMU部件，惯性测量传感器 -->
@@ -18,4 +19,18 @@
                 </material>
             </visual>
+            <collision>
+                <!-- 沿着自己几何中心的偏移和旋转 -->
+                <origin xyz="0.0 0.0 0.0" rpy="0.0 0.0 0.0"/>
+                <!-- 几何形状 -->
+                <geometry>
+                    <!-- 圆柱体 radius 半径 0.10m  高度 0.12m-->
+                    <box size="0.02 0.02 0.02"/>
+                </geometry>
+                <!-- 材质颜色 -->
+                <material name="black">
+                    <color rgba="0.0 0.0 0.0 0.5"/>
+                </material>
+            </collision>
+            <xacro:box_inertia m="0.05" w="0.02" h="0.02" d="0.02" />
         </link>
         <!-- 机器人的关节，用于组合机器人的部件 -->

File: Simulation/sim_ws/src/duanbot_description/urdf/duanbot/sensor/laser.urdf.xacro (robot description, xacro)
@@ -1,4 +1,5 @@
 <?xml version="1.0"?>
 <robot xmlns:xacro="http://www.ros.org/wiki/xacro">
+<xacro:include filename="$(find duanbot_description)/urdf/duanbot/common_inertia.xacro"/>
     <xacro:macro name="laser_xacro" params="xyz">
         <!-- 雷达支撑杆 -->
@@ -18,4 +19,18 @@
                 </material>
             </visual>
+            <collision>
+                <!-- 沿着自己几何中心的偏移和旋转 -->
+                <origin xyz="0.0 0.0 0.0" rpy="0.0 0.0 0.0"/>
+                <!-- 几何形状 -->
+                <geometry>
+                    <!-- 圆柱体 radius 半径 0.10m  高度 0.12m-->
+                    <cylinder radius="0.01" length="0.10"/>
+                </geometry>
+                <!-- 材质颜色 -->
+                <material name="black">
+                    <color rgba="0.0 0.0 0.0 1.0"/>
+                </material>
+            </collision>
+            <xacro:cylinder_inertia m="0.05" r="0.01" h="0.10" />
         </link>
         <!-- 雷达 -->
@@ -35,4 +50,18 @@
                 </material>
             </visual>
+            <collision>
+                <!-- 沿着自己几何中心的偏移和旋转 -->
+                <origin xyz="0.0 0.0 0.0" rpy="0.0 0.0 0.0"/>
+                <!-- 几何形状 -->
+                <geometry>
+                    <!-- 圆柱体 radius 半径 0.10m  高度 0.12m-->
+                    <cylinder radius="0.02" length="0.02"/>
+                </geometry>
+                <!-- 材质颜色 -->
+                <material name="black">
+                    <color rgba="0.0 0.0 0.0 1.0"/>
+                </material>
+            </collision>
+            <xacro:cylinder_inertia m="0.10" r="0.02" h="0.02" />
         </link>
         <joint name="laser_joint" type="fixed">
@@ -46,4 +75,10 @@
             <origin xyz="${xyz}" rpy="0.0 0.0 0.0"/>
         </joint>
+        <gazebo reference="laser_cylinder_link">
+            <material>Gazebo/Black</material>
+        </gazebo>
+        <gazebo reference="laser_link">
+            <material>Gazebo/Black</material>
+        </gazebo>
     </xacro:macro>
 </robot>
