Commit message: navigation

File: duan-src/duan_ws/src/duanbot_description/urdf/duanbot/sensor/imu.urdf.xacro (robot description, xacro)
@@ -2,6 +2,7 @@
 <robot xmlns:xacro="http://www.ros.org/wiki/xacro">
 <xacro:include filename="$(find duanbot_description)/urdf/duanbot/common_inertia.xacro"/>
-    <xacro:macro name="camera_xacro" params="xyz">
-        <link name="camera_link">
+    <xacro:macro name="imu_xacro" params="xyz">
+        <!-- 机器人的IMU部件，惯性测量传感器 -->
+        <link name="imu_link">
             <!-- 部件的外观描述 -->
             <visual>
@@ -10,5 +11,6 @@
                 <!-- 几何形状 -->
                 <geometry>
-                    <box size="0.02 0.10 0.02"/>
+                    <!-- 圆柱体 radius 半径 0.10m  高度 0.12m-->
+                    <box size="0.02 0.02 0.02"/>
                 </geometry>
                 <!-- 材质颜色 -->
@@ -22,5 +24,6 @@
                 <!-- 几何形状 -->
                 <geometry>
-                    <box size="0.02 0.10 0.02"/>
+                    <!-- 圆柱体 radius 半径 0.10m  高度 0.12m-->
+                    <box size="0.02 0.02 0.02"/>
                 </geometry>
                 <!-- 材质颜色 -->
@@ -29,18 +32,11 @@
                 </material>
             </collision>
-            <xacro:box_inertia m="0.1" w="0.02" h="0.10" d="0.02" />
+            <xacro:box_inertia m="0.05" w="0.02" h="0.02" d="0.02" />
         </link>
-        <link name="camera_optical_link"></link>
         <!-- 机器人的关节，用于组合机器人的部件 -->
-        <joint name="camera_joint" type="fixed">
+        <joint name="imu_joint" type="fixed">
             <parent link="base_link"/>
-            <child link="camera_link"/>
+            <child link="imu_link"/>
             <origin xyz="${xyz}" rpy="0.0 0.0 0.0"/>
-        </joint>
-        <!-- 这里目的是做一个修正 让相机z轴朝前方 -->
-        <joint name="camera_optical_joint" type="fixed">
-            <parent link="camera_link"/>
-            <child link="camera_optical_link"/>
-            <origin xyz="0 0 0" rpy="${-pi/2} 0.0 0.0"/>
         </joint>
     </xacro:macro>
